File: KiCad/Template/opencamera-default/connectors.sch (KiCad schematic (older format))
At the start: 4 parts, among them P1 CONN_LEFT_TOP, P2 CONN_RIGHT_TOP, P3 CONN_LEFT_BOTTOM, P4 CONN_RIGHT_BOTTOM

Commit message: Update Template
v1.1
Removed keepouts around mounting holes (looks nicer).
Modified board-board connectors to include grounded mounting pads with
through via.
Created test point footprints.
Added 1,2,3,4 layer text to confirm proper stackup when receiving from
fab.
Parts:
- removed P1: CONN_LEFT_TOP, OpenCamera:DF17_60_RECEPTACLE, symbol CONN_02X30
- removed P2: CONN_RIGHT_TOP, OpenCamera:DF17_60_RECEPTACLE, symbol CONN_02X30
- removed P3: CONN_LEFT_BOTTOM, OpenCamera:DF17_60_HEADER, symbol CONN_02X30
- removed P4: CONN_RIGHT_BOTTOM, OpenCamera:DF17_60_HEADER, symbol CONN_02X30
- added P1: CONN_LEFT_TOP, symbol CONN_02X31
- added P2: CONN_RIGHT_TOP, symbol CONN_02X31
- added P3: CONN_LEFT_BOTTOM, symbol CONN_02X31
- added P4: CONN_RIGHT_BOTTOM, symbol CONN_02X31
Connections:
- wire segments 248 -> 256
Changed lines of the file:
@@
 LIBS:valves
 LIBS:OpenCamera
-LIBS:Template-cache
 EELAYER 25 0
 EELAYER END
@@
 Sheet 2 2
 Title "Board-Board Connectors"
-Date "Sunday, June 07, 2015"
-Rev "v1.0"
+Date "Saturday, June 13, 2015"
+Rev "1.1"
 Comp "Open Camera Project"
 Comment1 "Author: Brian Schiffer"
@@
 Comment4 ""
 $EndDescr
-$Comp
-L CONN_02X30 P1
-U 1 1 55749249
-P 1250 3900
-F 0 "P1" H 1250 5450 50  0000 C CNN
-F 1 "CONN_LEFT_TOP" V 1250 3900 50  0000 C CNN
-F 2 "OpenCamera:DF17_60_RECEPTACLE" H 1250 3400 60  0001 C CNN
-F 3 "" H 1250 3400 60  0000 C CNN
-	1    1250 3900
-	1    0    0    -1
-$EndComp
-$Comp
-L CONN_02X30 P3
-U 1 1 557492B9
-P 2250 3900
-F 0 "P3" H 2250 5450 50  0000 C CNN
-F 1 "CONN_LEFT_BOTTOM" V 2250 3900 50  0000 C CNN
-F 2 "OpenCamera:DF17_60_HEADER" H 2250 3400 60  0001 C CNN
-F 3 "" H 2250 3400 60  0000 C CNN
-	1    2250 3900
-	1    0    0    -1
-$EndComp
-$Comp
-L CONN_02X30 P4
-U 1 1 557492FE
-P 8750 3900
-F 0 "P4" H 8750 5450 50  0000 C CNN
-F 1 "CONN_RIGHT_BOTTOM" V 8750 3900 50  0000 C CNN
-F 2 "OpenCamera:DF17_60_HEADER" H 8750 3400 60  0001 C CNN
-F 3 "" H 8750 3400 60  0000 C CNN
-	1    8750 3900
-	1    0    0    -1
-$EndComp
-$Comp
-L CONN_02X30 P2
-U 1 1 55749341
-P 9750 3900
-F 0 "P2" H 9750 5450 50  0000 C CNN
-F 1 "CONN_RIGHT_TOP" V 9750 3900 50  0000 C CNN
-F 2 "OpenCamera:DF17_60_RECEPTACLE" H 9750 3400 60  0001 C CNN
-F 3 "" H 9750 3400 60  0000 C CNN
-	1    9750 3900
-	1    0    0    -1
-$EndComp
 Wire Wire Line
 	1500 2450 2000 2450
@@
 L GNDD #PWR01
 U 1 1 5574A4C4
-P 950 5450
-F 0 "#PWR01" H 950 5200 50  0001 C CNN
-F 1 "GNDD" H 950 5300 50  0000 C CNN
-F 2 "" H 950 5450 60  0000 C CNN
-F 3 "" H 950 5450 60  0000 C CNN
-	1    950  5450
+P 950 5550
+F 0 "#PWR01" H 950 5300 50  0001 C CNN
+F 1 "GNDD" H 950 5400 50  0000 C CNN
+F 2 "" H 950 5550 60  0000 C CNN
+F 3 "" H 950 5550 60  0000 C CNN
+	1    950  5550
 	1    0    0    -1
 $EndComp
@@
 L GNDD #PWR02
 U 1 1 5574A4DC
-P 2550 5450
-F 0 "#PWR02" H 2550 5200 50  0001 C CNN
-F 1 "GNDD" H 2550 5300 50  0000 C CNN
-F 2 "" H 2550 5450 60  0000 C CNN
-F 3 "" H 2550 5450 60  0000 C CNN
-	1    2550 5450
+P 2550 5550
+F 0 "#PWR02" H 2550 5300 50  0001 C CNN
+F 1 "GNDD" H 2550 5400 50  0000 C CNN
+F 2 "" H 2550 5550 60  0000 C CNN
+F 3 "" H 2550 5550 60  0000 C CNN
+	1    2550 5550
 	1    0    0    -1
 $EndComp
@@
 L GNDA #PWR03
 U 1 1 5574A4F4
-P 8450 5450
-F 0 "#PWR03" H 8450 5200 50  0001 C CNN
-F 1 "GNDA" H 8450 5300 50  0000 C CNN
-F 2 "" H 8450 5450 60  0000 C CNN
-F 3 "" H 8450 5450 60  0000 C CNN
-	1    8450 5450
+P 8450 5550
+F 0 "#PWR03" H 8450 5300 50  0001 C CNN
+F 1 "GNDA" H 8450 5400 50  0000 C CNN
+F 2 "" H 8450 5550 60  0000 C CNN
+F 3 "" H 8450 5550 60  0000 C CNN
+	1    8450 5550
 	1    0    0    -1
 $EndComp
@@
 L GNDA #PWR04
 U 1 1 5574A50C
-P 10050 5450
-F 0 "#PWR04" H 10050 5200 50  0001 C CNN
-F 1 "GNDA" H 10050 5300 50  0000 C CNN
-F 2 "" H 10050 5450 60  0000 C CNN
-F 3 "" H 10050 5450 60  0000 C CNN
-	1    10050 5450
+P 10050 5550
+F 0 "#PWR04" H 10050 5300 50  0001 C CNN
+F 1 "GNDA" H 10050 5400 50  0000 C CNN
+F 2 "" H 10050 5550 60  0000 C CNN
+F 3 "" H 10050 5550 60  0000 C CNN
+	1    10050 5550
 	1    0    0    -1
 $EndComp
@@
 	1000 2450 950  2450
 Wire Wire Line
-	950  2450 950  5450
+	950  2450 950  5550
 Wire Wire Line
 	2500 2450 2550 2450
 Wire Wire Line
-	2550 2450 2550 5450
+	2550 2450 2550 5550
 Wire Wire Line
 	1000 2550 950  2550
@@
 	8500 2450 8450 2450
 Wire Wire Line
-	8450 2450 8450 5450
+	8450 2450 8450 5550
 Wire Wire Line
 	10000 2450 10050 2450
 Wire Wire Line
-	10050 2450 10050 5450
+	10050 2450 10050 5550
 Wire Wire Line
 	8500 2550 8450 2550
@@
 Text Label 6000 5350 2    60   ~ 0
 R30
+$Comp
+L CONN_02X31 P1
+U 1 1 557C3923
+P 1250 3950
+F 0 "P1" H 1250 5550 50  0000 C CNN
+F 1 "CONN_LEFT_TOP" V 1250 3950 50  0000 C CNN
+F 2 "" H 1250 3500 60  0000 C CNN
+F 3 "" H 1250 3500 60  0000 C CNN
+	1    1250 3950
+	1    0    0    -1
+$EndComp
+$Comp
+L CONN_02X31 P3
+U 1 1 557C3BC1
+P 2250 3950
+F 0 "P3" H 2250 5550 50  0000 C CNN
+F 1 "CONN_LEFT_BOTTOM" V 2250 3950 50  0000 C CNN
+F 2 "" H 2250 3500 60  0000 C CNN
+F 3 "" H 2250 3500 60  0000 C CNN
+	1    2250 3950
+	1    0    0    -1
+$EndComp
+Wire Wire Line
+	1000 5450 950  5450
+Connection ~ 950  5450
+Wire Wire Line
+	2500 5450 2550 5450
+Connection ~ 2550 5450
+Wire Wire Line
+	1500 5450 2000 5450
+$Comp
+L GNDD #PWR07
+U 1 1 557C43E8
+P 1750 5550
+F 0 "#PWR07" H 1750 5300 50  0001 C CNN
+F 1 "GNDD" H 1750 5400 50  0000 C CNN
+F 2 "" H 1750 5550 60  0000 C CNN
+F 3 "" H 1750 5550 60  0000 C CNN
+	1    1750 5550
+	1    0    0    -1
+$EndComp
+Wire Wire Line
+	1750 5550 1750 5450
+Connection ~ 1750 5450
+$Comp
+L CONN_02X31 P4
+U 1 1 557C4BF1
+P 8750 3950
+F 0 "P4" H 8750 5550 50  0000 C CNN
+F 1 "CONN_RIGHT_BOTTOM" V 8750 3950 50  0000 C CNN
+F 2 "" H 8750 3500 60  0000 C CNN
+F 3 "" H 8750 3500 60  0000 C CNN
+	1    8750 3950
+	1    0    0    -1
+$EndComp
+$Comp
+L CONN_02X31 P2
+U 1 1 557C4C8A
+P 9750 3950
+F 0 "P2" H 9750 5550 50  0000 C CNN
+F 1 "CONN_RIGHT_TOP" V 9750 3950 50  0000 C CNN
+F 2 "" H 9750 3500 60  0000 C CNN
+F 3 "" H 9750 3500 60  0000 C CNN
+	1    9750 3950
+	1    0    0    -1
+$EndComp
+Wire Wire Line
+	8500 5450 8450 5450
+Connection ~ 8450 5450
+Wire Wire Line
+	9000 5450 9500 5450
+Wire Wire Line
+	10000 5450 10050 5450
+Connection ~ 10050 5450
+$Comp
+L GNDA #PWR08
+U 1 1 557C5306
+P 9250 5550
+F 0 "#PWR08" H 9250 5300 50  0001 C CNN
+F 1 "GNDA" H 9250 5400 50  0000 C CNN
+F 2 "" H 9250 5550 60  0000 C CNN
+F 3 "" H 9250 5550 60  0000 C CNN
+	1    9250 5550
+	1    0    0    -1
+$EndComp
+Wire Wire Line
+	9250 5550 9250 5450
+Connection ~ 9250 5450
 $EndSCHEMATC
