File: KiCad/Debug_Board/v1.0/Debug_Board.sch (KiCad schematic (older format))
At the start: 3 parts, among them P5 CONN_02X30, P6 CONN_02X01, P7 CONN_02X30

Commit message: Power board started
Created some schematic symbols for power board parts.
Also, started the hierarchy sheets.
Parts:
- P5, P7: footprint (none) -> OpenCamera:CONN60_RIGHT_ANGLE
- P6: footprint (none) -> OpenCamera:CONN2_RIGHT_ANGLE
Changed lines of the file:
@@
 F 0 "P7" H 6150 5000 50  0000 C CNN
 F 1 "CONN_02X30" V 6150 3450 50  0000 C CNN
-F 2 "" H 6150 2950 60  0000 C CNN
+F 2 "OpenCamera:CONN60_RIGHT_ANGLE" H 6150 2950 60  0001 C CNN
 F 3 "" H 6150 2950 60  0000 C CNN
 	1    6150 3450
@@
 F 0 "P5" H 4500 5000 50  0000 C CNN
 F 1 "CONN_02X30" V 4500 3450 50  0000 C CNN
-F 2 "" H 4500 2950 60  0000 C CNN
+F 2 "OpenCamera:CONN60_RIGHT_ANGLE" H 4500 2950 60  0001 C CNN
 F 3 "" H 4500 2950 60  0000 C CNN
 	1    4500 3450
@@
 	5750 4900 5900 4900
 $Comp
-L GNDA #PWR4
+L GNDA #PWR01
 U 1 1 557756EB
 P 6500 5100
-F 0 "#PWR4" H 6500 4850 50  0001 C CNN
+F 0 "#PWR01" H 6500 4850 50  0001 C CNN
 F 1 "GNDA" H 6500 4950 50  0000 C CNN
 F 2 "" H 6500 5100 60  0000 C CNN
@@
 $EndComp
 $Comp
-L GNDD #PWR1
+L GNDD #PWR02
 U 1 1 55775D9B
 P 4200 5100
-F 0 "#PWR1" H 4200 4850 50  0001 C CNN
+F 0 "#PWR02" H 4200 4850 50  0001 C CNN
 F 1 "GNDD" H 4200 4950 50  0000 C CNN
 F 2 "" H 4200 5100 60  0000 C CNN
@@
 F 0 "P6" H 5300 950 50  0000 C CNN
 F 1 "CONN_02X01" H 5300 750 50  0000 C CNN
-F 2 "" H 5300 -350 60  0000 C CNN
+F 2 "OpenCamera:CONN2_RIGHT_ANGLE" H 5300 -350 60  0001 C CNN
 F 3 "" H 5300 -350 60  0000 C CNN
 	1    5300 850
@@
 $EndComp
 $Comp
-L GNDA #PWR3
+L GNDA #PWR03
 U 1 1 557826FF
 P 5650 1000
-F 0 "#PWR3" H 5650 750 50  0001 C CNN
+F 0 "#PWR03" H 5650 750 50  0001 C CNN
 F 1 "GNDA" H 5650 850 50  0000 C CNN
 F 2 "" H 5650 1000 60  0000 C CNN
@@
 $EndComp
 $Comp
-L GNDD #PWR2
+L GNDD #PWR04
 U 1 1 557827D0
 P 4950 1000
-F 0 "#PWR2" H 4950 750 50  0001 C CNN
+F 0 "#PWR04" H 4950 750 50  0001 C CNN
 F 1 "GNDD" H 4950 850 50  0000 C CNN
 F 2 "" H 4950 1000 60  0000 C CNN
