File: KiCad/Power_Board/connectors.sch (KiCad schematic (older format))
At the start: 4 parts, among them P1 CONN_LEFT_TOP, P2 CONN_RIGHT_TOP, P3 CONN_LEFT_BOTTOM, P4 CONN_RIGHT_BOTTOM

Commit message: Linked footprints to schematic.
Also cleaned up some footprint errors:
Changed IC footprint names to be invisible on the silkscreen layer.
Fixed test points that were lacking pin numbers causing netlist
failures.
Parts:
- P1, P2: footprint (none) -> OpenCamera:DF17_60_RECEPTACLE
- P3, P4: footprint (none) -> OpenCamera:DF17_60_HEADER
Changed lines of the file:
@@
 	9000 5350 9500 5350
 $Comp
-L GNDD #PWR12
+L GNDD #PWR012
 U 1 1 5574A4C4
 P 950 5550
-F 0 "#PWR12" H 950 5300 50  0001 C CNN
+F 0 "#PWR012" H 950 5300 50  0001 C CNN
 F 1 "GNDD" H 950 5400 50  0000 C CNN
 F 2 "" H 950 5550 60  0000 C CNN
@@
 $EndComp
 $Comp
-L GNDD #PWR14
+L GNDD #PWR013
 U 1 1 5574A4DC
 P 2550 5550
-F 0 "#PWR14" H 2550 5300 50  0001 C CNN
+F 0 "#PWR013" H 2550 5300 50  0001 C CNN
 F 1 "GNDD" H 2550 5400 50  0000 C CNN
 F 2 "" H 2550 5550 60  0000 C CNN
@@
 $EndComp
 $Comp
-L GNDA #PWR17
+L GNDA #PWR014
 U 1 1 5574A4F4
 P 8450 5550
-F 0 "#PWR17" H 8450 5300 50  0001 C CNN
+F 0 "#PWR014" H 8450 5300 50  0001 C CNN
 F 1 "GNDA" H 8450 5400 50  0000 C CNN
 F 2 "" H 8450 5550 60  0000 C CNN
@@
 $EndComp
 $Comp
-L GNDA #PWR19
+L GNDA #PWR015
 U 1 1 5574A50C
 P 10050 5550
-F 0 "#PWR19" H 10050 5300 50  0001 C CNN
+F 0 "#PWR015" H 10050 5300 50  0001 C CNN
 F 1 "GNDA" H 10050 5400 50  0000 C CNN
 F 2 "" H 10050 5550 60  0000 C CNN
@@
 L30
 $Comp
-L GNDD #PWR15
+L GNDD #PWR016
 U 1 1 557535BD
 P 5000 5500
-F 0 "#PWR15" H 5000 5250 50  0001 C CNN
+F 0 "#PWR016" H 5000 5250 50  0001 C CNN
 F 1 "GNDD" H 5000 5350 50  0000 C CNN
 F 2 "" H 5000 5500 60  0000 C CNN
@@
 	6200 5450 6000 5450
 $Comp
-L GNDA #PWR16
+L GNDA #PWR017
 U 1 1 557564C2
 P 6000 5500
-F 0 "#PWR16" H 6000 5250 50  0001 C CNN
+F 0 "#PWR017" H 6000 5250 50  0001 C CNN
 F 1 "GNDA" H 6000 5350 50  0000 C CNN
 F 2 "" H 6000 5500 60  0000 C CNN
@@
 F 0 "P1" H 1250 5550 50  0000 C CNN
 F 1 "CONN_LEFT_TOP" V 1250 3950 50  0000 C CNN
-F 2 "" H 1250 3500 60  0000 C CNN
+F 2 "OpenCamera:DF17_60_RECEPTACLE" H 1250 3500 60  0001 C CNN
 F 3 "" H 1250 3500 60  0000 C CNN
 	1    1250 3950
@@
 F 0 "P3" H 2250 5550 50  0000 C CNN
 F 1 "CONN_LEFT_BOTTOM" V 2250 3950 50  0000 C CNN
-F 2 "" H 2250 3500 60  0000 C CNN
+F 2 "OpenCamera:DF17_60_HEADER" H 2250 3500 60  0001 C CNN
 F 3 "" H 2250 3500 60  0000 C CNN
 	1    2250 3950
@@
 	1500 5450 2000 5450
 $Comp
-L GNDD #PWR13
+L GNDD #PWR018
 U 1 1 557C43E8
 P 1750 5550
-F 0 "#PWR13" H 1750 5300 50  0001 C CNN
+F 0 "#PWR018" H 1750 5300 50  0001 C CNN
 F 1 "GNDD" H 1750 5400 50  0000 C CNN
 F 2 "" H 1750 5550 60  0000 C CNN
@@
 F 0 "P4" H 8750 5550 50  0000 C CNN
 F 1 "CONN_RIGHT_BOTTOM" V 8750 3950 50  0000 C CNN
-F 2 "" H 8750 3500 60  0000 C CNN
+F 2 "OpenCamera:DF17_60_HEADER" H 8750 3500 60  0001 C CNN
 F 3 "" H 8750 3500 60  0000 C CNN
 	1    8750 3950
@@
 F 0 "P2" H 9750 5550 50  0000 C CNN
 F 1 "CONN_RIGHT_TOP" V 9750 3950 50  0000 C CNN
-F 2 "" H 9750 3500 60  0000 C CNN
+F 2 "OpenCamera:DF17_60_RECEPTACLE" H 9750 3500 60  0001 C CNN
 F 3 "" H 9750 3500 60  0000 C CNN
 	1    9750 3950
@@
 Connection ~ 10050 5450
 $Comp
-L GNDA #PWR18
+L GNDA #PWR019
 U 1 1 557C5306
 P 9250 5550
-F 0 "#PWR18" H 9250 5300 50  0001 C CNN
+F 0 "#PWR019" H 9250 5300 50  0001 C CNN
 F 1 "GNDA" H 9250 5400 50  0000 C CNN
 F 2 "" H 9250 5550 60  0000 C CNN
