File: KiCad/Power_Board/Analog_Power.sch (KiCad schematic (older format))
At the start: 69 parts, among them P10 CONN_02X01, P8 CONN_02X01, P9 CONN_02X01, Q1 IRLL024NQ, U10 ADP7142_CSP, U11 ADP7182_CSP, U12 ADP3335_CSP, U7 MAX152x, U8 ADP5070, U9 TPS63030

Commit message: Component changes
Switched Vref test point to test clip.
Beefed up 0ohm jumpers to 0805.
Parts:
- R22, R23, R30, R31, R32: footprint Resistors_SMD:R_0402 -> Resistors_SMD:R_0805
Changed lines of the file:
@@
 F 0 "R22" V 5100 1250 50  0000 L CNN
 F 1 "0" V 5300 1250 50  0000 L CNN
-F 2 "Resistors_SMD:R_0402" H 5200 1300 60  0001 C CNN
+F 2 "Resistors_SMD:R_0805" H 5200 1300 60  0001 C CNN
 F 3 "" H 5200 1300 60  0000 C CNN
 	1    5200 1300
@@
 F 0 "R30" V 7950 1250 50  0000 L CNN
 F 1 "0" V 8150 1250 50  0000 L CNN
-F 2 "Resistors_SMD:R_0402" H 8050 1300 60  0001 C CNN
+F 2 "Resistors_SMD:R_0805" H 8050 1300 60  0001 C CNN
 F 3 "" H 8050 1300 60  0000 C CNN
 	1    8050 1300
@@
 F 0 "R23" V 5750 5850 50  0000 L CNN
 F 1 "0" V 5950 5850 50  0000 L CNN
-F 2 "Resistors_SMD:R_0402" H 5850 5900 60  0001 C CNN
+F 2 "Resistors_SMD:R_0805" H 5850 5900 60  0001 C CNN
 F 3 "" H 5850 5900 60  0000 C CNN
 	1    5850 5900
@@
 F 0 "R32" V 8850 4100 50  0000 L CNN
 F 1 "0" V 9050 4100 50  0000 L CNN
-F 2 "Resistors_SMD:R_0402" H 8950 4150 60  0001 C CNN
+F 2 "Resistors_SMD:R_0805" H 8950 4150 60  0001 C CNN
 F 3 "" H 8950 4150 60  0000 C CNN
 	1    8950 4150
@@
 F 0 "R31" V 8850 3000 50  0000 L CNN
 F 1 "0" V 9050 3000 50  0000 L CNN
-F 2 "Resistors_SMD:R_0402" H 8950 3050 60  0001 C CNN
+F 2 "Resistors_SMD:R_0805" H 8950 3050 60  0001 C CNN
 F 3 "" H 8950 3050 60  0000 C CNN
 	1    8950 3050

Commit message: Initialized Driver Board Schematic & PCB from template
(also updated power board for the kicad version on my new computer)
Parts:
- D1, D3, D4: symbol D_Schottky_Small -> D_Schottky_Small-RESCUE-Power_Board
- D2: symbol D_Small -> D_Small-RESCUE-Power_Board
- Q1: symbol Q_NMOS_GDSD -> Q_NMOS_GDSD-RESCUE-Power_Board
Changed lines of the file:
@@
 EESchema Schematic File Version 2
+LIBS:Power_Board-rescue
 LIBS:power
 LIBS:device
@@
 LIBS:memory
 LIBS:xilinx
-LIBS:special
 LIBS:microcontrollers
 LIBS:dsp
@@
 $EndComp
 $Comp
-L D_Schottky_Small D3
+L D_Schottky_Small-RESCUE-Power_Board D3
 U 1 1 55907FA3
 P 4300 3050
@@
 $EndComp
 $Comp
-L D_Schottky_Small D1
+L D_Schottky_Small-RESCUE-Power_Board D1
 U 1 1 559083A5
 P 3800 4150
@@
 $EndComp
 $Comp
-L Q_NMOS_GDSD Q1
+L Q_NMOS_GDSD-RESCUE-Power_Board Q1
 U 1 1 5592DB19
 P 3250 6200
@@
 $EndComp
 $Comp
-L D_Schottky_Small D4
+L D_Schottky_Small-RESCUE-Power_Board D4
 U 1 1 5592DF1A
 P 4400 6500
@@
 	2150 5900 1700 5900
 $Comp
-L D_Small D2
+L D_Small-RESCUE-Power_Board D2
 U 1 1 5592F334
 P 4100 5900
